Commit message: 关闭随机化

File: resources/robots/F2_ZZ1_waiguan/x3_f2_14dof.urdf (robot description, URDF)
Before this commit: robot F2, 46 links, 45 joints
Links:
- link left_ankle_roll_link: geometry collision capsule length=0.100 radius=0.01; collision capsule length=0.100 radius=0.01
- link right_ankle_roll_link: geometry collision capsule length=0.100 radius=0.01; collision capsule length=0.100 radius=0.01
